Commit message: improve slam and add octomap

File: drone_test/urdf/x500.urdf (robot description, URDF)
Before this commit: robot x500_drone, 8 links, 7 joints
Links:
- removed link dummy_root
Joints:
- removed joint dummy_joint

Commit message: using lidar, octomap is working

File: drone_test/urdf/x500.urdf (robot description, URDF)
Before this commit: robot x500_drone, 7 links, 6 joints
Links:
- added link lidar_link; visual cylinder length=0.04 radius=0.03
Joints:
- added joint lidar_joint: type fixed, parent base_link, child lidar_link, origin xyz=0 0 0.12 rpy=0 0 0
