Commit message: add nav, add main (correct)

File: drone_main/urdf/x500.urdf (robot description, URDF)
Before this commit: robot x500_drone, 8 links, 7 joints
Links:
- link base_link: geometry collision box size=0.015 0.015 0.21; collision box size=0.015 0.015 0.21
- link rotor_0: geometry collision box size=0.279 0.016 0.0008; visual mesh filename=package://drone_main/meshes/1345_prop_ccw.stl scale=0.846 0.846 0.846
- link rotor_1: geometry collision box size=0.279 0.016 0.0008; visual mesh filename=package://drone_main/meshes/1345_prop_ccw.stl scale=0.846 0.846 0.846
- link rotor_2: geometry collision box size=0.279 0.016 0.0008; visual mesh filename=package://drone_main/meshes/1345_prop_cw.stl scale=0.846 0.846 0.846
- link rotor_3: geometry collision box size=0.279 0.016 0.0008; visual mesh filename=package://drone_main/meshes/1345_prop_cw.stl scale=0.846 0.846 0.846

Commit message: add README, upload package.xml and add first version of human follow

File: drone_main/urdf/x500.urdf (robot description, URDF)
Before this commit: robot x500_drone, 8 links, 7 joints
Joints:
- joint camera_joint: origin xyz=0.18 0 0.05 rpy=0 0 0 -> xyz=0.18 0 0.05 rpy=0 0.349 0
