Commit message: check position camera and lidar

File: drone_main/urdf/x500.urdf (robot description, URDF)
Before this commit: robot x500_drone, 8 links, 7 joints
Links:
- link lidar_link: geometry visual cylinder length=0.02 radius=0.01
Joints:
- joint camera_joint: origin xyz=0.18 0 0.05 rpy=0 0.349 0 -> xyz=0.17 0 -0.01 rpy=0 0.349 0
- joint lidar_joint: origin xyz=0 0 0.12 rpy=0 0 0 -> xyz=0 0 0.065 rpy=0 0 0
